File: Hardware/VeinCamHat/VeinCamHat.sch (KiCad schematic (older format))
At the start: 23 parts, among them J1 Raspberry_Pi_2_3, Q1 NTJD4001N

Commit message: updating hardware things
Connections:
- net GND: no longer R2.2
- net nLED_BOOT: no longer D2.1 (K)
- new net: D2.1 (K), R2.2
Other:
- moved on the sheet: D2, R2
Changed lines of the file:
@@
 L Device:R R2
 U 1 1 5D6666C3
-P 4100 2800
-F 0 "R2" H 4150 2850 50  0000 L CNN
-F 1 "1K5" H 4150 2750 50  0000 L CNN
-F 2 "Resistor_SMD:R_0603_1608Metric" V 4030 2800 50  0001 C CNN
-F 3 "~" H 4100 2800 50  0001 C CNN
-	1    4100 2800
-	1    0    0    -1
+P 4150 2550
+F 0 "R2" V 4225 2500 50  0000 L CNN
+F 1 "1K5" V 4050 2475 50  0000 L CNN
+F 2 "Resistor_SMD:R_0603_1608Metric" V 4080 2550 50  0001 C CNN
+F 3 "~" H 4150 2550 50  0001 C CNN
+	1    4150 2550
+	0    -1   -1   0
 $EndComp
 $Comp
 L Device:LED D2
 U 1 1 5D6666CA
-P 4400 2550
-F 0 "D2" H 4450 2650 50  0000 R CNN
-F 1 "RED LED" H 4650 2450 50  0000 R CNN
-F 2 "LED_SMD:LED_0805_2012Metric" H 4400 2550 50  0001 C CNN
-F 3 "~" H 4400 2550 50  0001 C CNN
-	1    4400 2550
+P 4550 2550
+F 0 "D2" H 4600 2650 50  0000 R CNN
+F 1 "RED LED" H 4800 2450 50  0000 R CNN
+F 2 "LED_SMD:LED_0805_2012Metric" H 4550 2550 50  0001 C CNN
+F 3 "~" H 4550 2550 50  0001 C CNN
+	1    4550 2550
 	1    0    0    -1
 $EndComp
@@
 	4900 2500 4900 2550
 Wire Wire Line
-	4550 2550 4900 2550
+	4700 2550 4900 2550
 Wire Wire Line
 	4700 1900 4900 1900
-Wire Wire Line
-	4100 2950 4100 3000
-$Comp
-L power:GND #PWR0104
-U 1 1 5CBB9F2E
-P 4100 3000
-F 0 "#PWR0104" H 4100 2750 50  0001 C CNN
-F 1 "GND" H 4105 2827 50  0000 C CNN
-F 2 "" H 4100 3000 50  0001 C CNN
-F 3 "" H 4100 3000 50  0001 C CNN
-	1    4100 3000
-	1    0    0    -1
-$EndComp
 $Comp
 L Connector:Raspberry_Pi_2_3 J1
@@
 Wire Wire Line
 	4300 1900 4400 1900
-Wire Wire Line
-	3500 2550 4100 2550
-Wire Wire Line
-	4100 2650 4100 2550
-Connection ~ 4100 2550
-Wire Wire Line
-	4100 2550 4250 2550
 NoConn ~ 1050 1650
 NoConn ~ 2650 2250
+Wire Wire Line
+	3500 2550 4000 2550
+Wire Wire Line
+	4300 2550 4400 2550
 $EndSCHEMATC

Commit message: Updates to board and generation of final production outputs
Parts:
- removed R3, R4, R5, R6: 3R3, Resistor_SMD:R_0603_1608Metric, symbol Device:R
- added RN1: R_Pack_3R3, Resistor_SMD:R_Array_Convex_4x0603, symbol Device:R_Pack04
Connections:
- net +5V: now also RN1.1 (R1.1), RN1.2 (R2.1), RN1.3 (R3.1), RN1.4 (R4.1)
- net at D3.2 (A2): now also RN1.8 (R1.2)
- net at D3.4 (A1): now also RN1.7 (R2.2)
- net at D4.2 (A2): now also RN1.5 (R4.2)
- net at D4.4 (A1): now also RN1.6 (R3.2)
Changed lines of the file:
@@
 Wire Wire Line
 	7850 2550 8200 2550
-Wire Wire Line
-	6300 2550 6150 2550
-Wire Wire Line
-	6300 2350 6150 2350
-Wire Wire Line
-	6300 1700 6150 1700
-Wire Wire Line
-	6300 1900 6150 1900
-Wire Wire Line
-	6100 2300 6150 2300
-Wire Wire Line
-	6150 2300 6150 2350
-Wire Wire Line
-	6150 2550 6150 2600
-Wire Wire Line
-	6150 2600 6100 2600
-$Comp
-L Device:R R3
-U 1 1 5C88BFEA
-P 5950 1650
-F 0 "R3" V 5850 1650 50  0000 C CNN
-F 1 "3R3" V 6050 1650 50  0000 C CNN
-F 2 "Resistor_SMD:R_0603_1608Metric" V 5880 1650 50  0001 C CNN
-F 3 "~" H 5950 1650 50  0001 C CNN
-	1    5950 1650
-	0    1    1    0
-$EndComp
-Wire Wire Line
-	6100 1950 6150 1950
-Wire Wire Line
-	6150 1950 6150 1900
-Wire Wire Line
-	6100 1650 6150 1650
-Wire Wire Line
-	6150 1650 6150 1700
-Wire Wire Line
-	5650 1500 5650 1650
-Wire Wire Line
-	5650 2600 5800 2600
-Wire Wire Line
-	5650 2300 5800 2300
-Connection ~ 5650 2300
-Wire Wire Line
-	5650 2300 5650 2600
-Wire Wire Line
-	5650 1950 5800 1950
-Connection ~ 5650 1950
-Wire Wire Line
-	5650 1950 5650 2300
-Wire Wire Line
-	5650 1650 5800 1650
-Connection ~ 5650 1650
-Wire Wire Line
-	5650 1650 5650 1950
 $Comp
 L power:+5V #PWR06
 U 1 1 5C8975EF
-P 5650 1500
-F 0 "#PWR06" H 5650 1350 50  0001 C CNN
-F 1 "+5V" H 5650 1640 50  0000 C CNN
-F 2 "" H 5650 1500 50  0000 C CNN
-F 3 "" H 5650 1500 50  0000 C CNN
-	1    5650 1500
+P 5500 1750
+F 0 "#PWR06" H 5500 1600 50  0001 C CNN
+F 1 "+5V" H 5500 1890 50  0000 C CNN
+F 2 "" H 5500 1750 50  0000 C CNN
+F 3 "" H 5500 1750 50  0000 C CNN
+	1    5500 1750
 	1    0    0    -1
 $EndComp
@@
 Text Notes 7300 1100 0    100  ~ 0
 IR LED's
-$Comp
-L Device:R R4
-U 1 1 5C8D8769
-P 5950 1950
-F 0 "R4" V 5850 1950 50  0000 C CNN
-F 1 "3R3" V 6050 1950 50  0000 C CNN
-F 2 "Resistor_SMD:R_0603_1608Metric" V 5880 1950 50  0001 C CNN
-F 3 "~" H 5950 1950 50  0001 C CNN
-	1    5950 1950
-	0    1    1    0
-$EndComp
-$Comp
-L Device:R R5
-U 1 1 5C8D87A7
-P 5950 2300
-F 0 "R5" V 5850 2300 50  0000 C CNN
-F 1 "3R3" V 6050 2300 50  0000 C CNN
-F 2 "Resistor_SMD:R_0603_1608Metric" V 5880 2300 50  0001 C CNN
-F 3 "~" H 5950 2300 50  0001 C CNN
-	1    5950 2300
-	0    1    1    0
-$EndComp
-$Comp
-L Device:R R6
-U 1 1 5C8D87E5
-P 5950 2600
-F 0 "R6" V 5850 2600 50  0000 C CNN
-F 1 "3R3" V 6050 2600 50  0000 C CNN
-F 2 "Resistor_SMD:R_0603_1608Metric" V 5880 2600 50  0001 C CNN
-F 3 "~" H 5950 2600 50  0001 C CNN
-	1    5950 2600
-	0    1    1    0
-$EndComp
 Wire Wire Line
 	10450 1700 10450 2350
@@
 Wire Wire Line
 	4300 2550 4400 2550
+Wire Wire Line
+	5550 2250 5500 2250
+Wire Wire Line
+	5500 2250 5500 2150
+Wire Wire Line
+	5500 1950 5550 1950
+Wire Wire Line
+	5550 2050 5500 2050
+Connection ~ 5500 2050
+Wire Wire Line
+	5500 2050 5500 1950
+Wire Wire Line
+	5550 2150 5500 2150
+Connection ~ 5500 2150
+Wire Wire Line
+	5500 2150 5500 2050
+Wire Wire Line
+	5500 1750 5500 1950
+Connection ~ 5500 1950
+Wire Wire Line
+	6050 1700 6300 1700
+$Comp
+L Device:R_Pack04 RN1
+U 1 1 5CEA12D3
+P 5750 2150
+F 0 "RN1" V 5333 2150 50  0000 C CNN
+F 1 "R_Pack_3R3" V 5424 2150 50  0000 C CNN
+F 2 "Resistor_SMD:R_Array_Convex_4x0603" V 6025 2150 50  0001 C CNN
+F 3 "~" H 5750 2150 50  0001 C CNN
+	1    5750 2150
+	0    1    1    0
+$EndComp
+Wire Wire Line
+	5950 2250 6150 2250
+Wire Wire Line
+	6150 2250 6150 2350
+Wire Wire Line
+	6150 2350 6300 2350
+Wire Wire Line
+	6050 2550 6050 2150
+Wire Wire Line
+	6050 2150 5950 2150
+Wire Wire Line
+	6050 2550 6300 2550
+Wire Wire Line
+	5950 1950 6050 1950
+Wire Wire Line
+	6050 1950 6050 1700
+Wire Wire Line
+	6150 2050 6150 1900
+Wire Wire Line
+	6150 1900 6300 1900
+Wire Wire Line
+	5950 2050 6150 2050
 $EndSCHEMATC
